File: ethernet-splitter.kicad_pcb (KiCad board)
At the start: 2 copper layers, 6 parts, among them J1 RJ45, J2 RJ45, J3 RJ45, J4 RJ45, J5 RJ45, U1 STM32F030C8Tx

Commit message: added de mux
Parts:
- added IC1: 74CBTLV3253PGG8, SamacSys_Parts:SOP65P640X120-16N, F.Cu at (141.0, 71.1)
- added IC2: 74CBTLV3253PGG8, SamacSys_Parts:SOP65P640X120-16N, F.Cu at (152.6, 76.6)
- added IC3: 74CBTLV3253PGG8, SamacSys_Parts:SOP65P640X120-16N, F.Cu at (142.4, 109.6)
- added IC4: 74CBTLV3253PGG8, SamacSys_Parts:SOP65P640X120-16N, F.Cu at (151.3, 109.6)
Connections:
- J5 pad 1: Net-(J4-Pad1) -> Net-(J5-Pad1)
- J5 pad 2: Net-(J4-Pad2) -> Net-(J5-Pad2)
- J5 pad 3: Net-(J4-Pad3) -> Net-(J5-Pad3)
- J5 pad 4: Net-(J4-Pad4) -> Net-(J5-Pad4)
- J5 pad 5: Net-(J4-Pad5) -> Net-(J5-Pad5)
- J5 pad 6: Net-(J4-Pad6) -> Net-(J5-Pad6)
- J5 pad 7: Net-(J4-Pad7) -> Net-(J5-Pad7)
- J5 pad 8: Net-(J4-Pad8) -> Net-(J5-Pad8)
