File: ethernet-splitter.sch (KiCad schematic (older format))
At the start: 6 parts, among them J1 RJ45, J2 RJ45, J3 RJ45, J4 RJ45, J5 RJ45, U1 STM32F030C8Tx

Commit message: Update ethernet-splitter.sch
Connections:
- net at J4.1: no longer J5.1
- net at J4.2: no longer J5.2
- net at J4.3: no longer J5.3
- net at J4.4: no longer J5.4
- net at J4.5: no longer J5.5
- net at J4.6: no longer J5.6
- net at J4.7: no longer J5.7
- net at J4.8: no longer J5.8
Changed lines of the file:
@@
 EESchema Schematic File Version 4
+LIBS:ethernet-splitter-cache
 EELAYER 29 0
 EELAYER END
@@
 	-1   0    0    1
 $EndComp
-Wire Wire Line
-	4400 4900 6250 4900
-Wire Wire Line
-	6250 4900 6250 4050
-Wire Wire Line
-	4400 5000 6200 5000
-Wire Wire Line
-	6200 5000 6200 3950
-Wire Wire Line
-	6200 3950 6250 3950
-Wire Wire Line
-	4400 5100 6150 5100
-Wire Wire Line
-	6150 5100 6150 3850
-Wire Wire Line
-	6150 3850 6250 3850
-Wire Wire Line
-	4400 5200 6100 5200
-Wire Wire Line
-	6100 5200 6100 3750
-Wire Wire Line
-	6100 3750 6250 3750
-Wire Wire Line
-	4400 5300 6050 5300
-Wire Wire Line
-	6050 5300 6050 3650
-Wire Wire Line
-	6050 3650 6250 3650
-Wire Wire Line
-	4400 5400 6000 5400
-Wire Wire Line
-	6000 5400 6000 3550
-Wire Wire Line
-	6000 3550 6250 3550
-Wire Wire Line
-	4400 5500 5950 5500
-Wire Wire Line
-	5950 5500 5950 3450
-Wire Wire Line
-	5950 3450 6250 3450
-Wire Wire Line
-	4400 5600 5900 5600
-Wire Wire Line
-	5900 5600 5900 3350
-Wire Wire Line
-	5900 3350 6250 3350
 $Comp
 L MCU_ST_STM32F0:STM32F030C8Tx U1

Commit message: added de mux
Parts:
- added IC1, IC2, IC3, IC4: 74CBTLV3253PGG8, SamacSys_Parts:SOP65P640X120-16N, symbol downloaded:74CBTLV3253PGG8
Other:
- moved on the sheet: J1, J2, J3, J4, J5, U1
Changed lines of the file:
@@
 L Connector:RJ45 J1
 U 1 1 62A6118C
-P 4000 2450
-F 0 "J1" H 3600 2550 50  0000 C CNN
-F 1 "RJ45" H 3600 2450 50  0000 C CNN
-F 2 "Connector_RJ:RJ45_Amphenol_54602-x08_Horizontal" V 4000 2475 50  0001 C CNN
-F 3 "~" V 4000 2475 50  0001 C CNN
-	1    4000 2450
+P 5050 2350
+F 0 "J1" H 4650 2450 50  0000 C CNN
+F 1 "RJ45" H 4650 2350 50  0000 C CNN
+F 2 "Connector_RJ:RJ45_Amphenol_54602-x08_Horizontal" V 5050 2375 50  0001 C CNN
+F 3 "~" V 5050 2375 50  0001 C CNN
+	1    5050 2350
 	1    0    0    -1
 $EndComp
@@
 L Connector:RJ45 J2
 U 1 1 62A6278C
-P 4000 3400
-F 0 "J2" H 3600 3500 50  0000 C CNN
-F 1 "RJ45" H 3600 3400 50  0000 C CNN
-F 2 "Connector_RJ:RJ45_Amphenol_54602-x08_Horizontal" V 4000 3425 50  0001 C CNN
-F 3 "~" V 4000 3425 50  0001 C CNN
-	1    4000 3400
+P 5050 3300
+F 0 "J2" H 4650 3400 50  0000 C CNN
+F 1 "RJ45" H 4650 3300 50  0000 C CNN
+F 2 "Connector_RJ:RJ45_Amphenol_54602-x08_Horizontal" V 5050 3325 50  0001 C CNN
+F 3 "~" V 5050 3325 50  0001 C CNN
+	1    5050 3300
 	1    0    0    -1
 $EndComp
@@
 L Connector:RJ45 J3
 U 1 1 62A64A11
-P 4000 4350
-F 0 "J3" H 3600 4450 50  0000 C CNN
-F 1 "RJ45" H 3600 4350 50  0000 C CNN
-F 2 "Connector_RJ:RJ45_Amphenol_54602-x08_Horizontal" V 4000 4375 50  0001 C CNN
-F 3 "~" V 4000 4375 50  0001 C CNN
-	1    4000 4350
+P 5050 4250
+F 0 "J3" H 4650 4350 50  0000 C CNN
+F 1 "RJ45" H 4650 4250 50  0000 C CNN
+F 2 "Connector_RJ:RJ45_Amphenol_54602-x08_Horizontal" V 5050 4275 50  0001 C CNN
+F 3 "~" V 5050 4275 50  0001 C CNN
+	1    5050 4250
 	1    0    0    -1
 $EndComp
@@
 L Connector:RJ45 J4
 U 1 1 62A66369
-P 4000 5300
-F 0 "J4" H 3600 5400 50  0000 C CNN
-F 1 "RJ45" H 3600 5300 50  0000 C CNN
-F 2 "Connector_RJ:RJ45_Amphenol_54602-x08_Horizontal" V 4000 5325 50  0001 C CNN
-F 3 "~" V 4000 5325 50  0001 C CNN
-	1    4000 5300
+P 5050 5200
+F 0 "J4" H 4650 5300 50  0000 C CNN
+F 1 "RJ45" H 4650 5200 50  0000 C CNN
+F 2 "Connector_RJ:RJ45_Amphenol_54602-x08_Horizontal" V 5050 5225 50  0001 C CNN
+F 3 "~" V 5050 5225 50  0001 C CNN
+	1    5050 5200
 	1    0    0    -1
 $EndComp
@@
 L Connector:RJ45 J5
 U 1 1 62A6BE13
-P 6650 3650
-F 0 "J5" H 6250 3750 50  0000 C CNN
-F 1 "RJ45" H 6250 3650 50  0000 C CNN
-F 2 "Connector_RJ:RJ45_Amphenol_54602-x08_Horizontal" V 6650 3675 50  0001 C CNN
-F 3 "~" V 6650 3675 50  0001 C CNN
-	1    6650 3650
+P 10350 2550
+F 0 "J5" H 9950 2650 50  0000 C CNN
+F 1 "RJ45" H 9950 2550 50  0000 C CNN
+F 2 "Connector_RJ:RJ45_Amphenol_54602-x08_Horizontal" V 10350 2575 50  0001 C CNN
+F 3 "~" V 10350 2575 50  0001 C CNN
+	1    10350 2550
 	-1   0    0    1
 $EndComp
@@
 L MCU_ST_STM32F0:STM32F030C8Tx U1
 U 1 1 62A75E3F
-P 8500 2850
-F 0 "U1" H 8500 1161 50  0000 C CNN
-F 1 "STM32F030C8Tx" H 8500 1070 50  0000 C CNN
-F 2 "Package_QFP:LQFP-48-1EP_7x7mm_P0.5mm_EP3.6x3.6mm" H 8000 1350 50  0001 R CNN
-F 3 "http://www.st.com/st-web-ui/static/active/en/resource/technical/document/datasheet/DM00088500.pdf" H 8500 2850 50  0001 C CNN
-	1    8500 2850
+P 1900 3800
+F 0 "U1" H 1900 2111 50  0000 C CNN
+F 1 "STM32F030C8Tx" H 1900 2020 50  0000 C CNN
+F 2 "Package_QFP:LQFP-48-1EP_7x7mm_P0.5mm_EP3.6x3.6mm" H 1400 2300 50  0001 R CNN
+F 3 "http://www.st.com/st-web-ui/static/active/en/resource/technical/document/datasheet/DM00088500.pdf" H 1900 3800 50  0001 C CNN
+	1    1900 3800
 	1    0    0    -1
 $EndComp
+$Comp
+L downloaded:74CBTLV3253PGG8 IC1
+U 1 1 62A6E752
+P 7000 2450
+F 0 "IC1" V 7504 2578 50  0000 L CNN
+F 1 "74CBTLV3253PGG8" V 7550 1750 50  0000 L CNN
+F 2 "SamacSys_Parts:SOP65P640X120-16N" H 7950 2550 50  0001 L CNN
+F 3 "https://componentsearchengine.com/Datasheets/1/74CBTLV3253PGG8.pdf" H 7950 2450 50  0001 L CNN
+F 4 "TSSOP 4.4 MM  0.65MM PITCH" H 7950 2350 50  0001 L CNN "Description"
+F 5 "1.2" H 7950 2250 50  0001 L CNN "Height"
+F 6 "972-74CBTLV3253PGG8" H 7950 2150 50  0001 L CNN "Mouser Part Number"
+F 7 "https://www.mouser.com/Search/Refine.aspx?Keyword=972-74CBTLV3253PGG8" H 7950 2050 50  0001 L CNN "Mouser Price/Stock"
+F 8 "IDT" H 7950 1950 50  0001 L CNN "Manufacturer_Name"
+F 9 "74CBTLV3253PGG8" H 7950 1850 50  0001 L CNN "Manufacturer_Part_Number"
+	1    7000 2450
+	0    1    1    0
+$EndComp
+$Comp
+L downloaded:74CBTLV3253PGG8 IC2
+U 1 1 62A70647
+P 7000 3850
+F 0 "IC2" V 7504 3978 50  0000 L CNN
+F 1 "74CBTLV3253PGG8" V 7550 3150 50  0000 L CNN
+F 2 "SamacSys_Parts:SOP65P640X120-16N" H 7950 3950 50  0001 L CNN
+F 3 "https://componentsearchengine.com/Datasheets/1/74CBTLV3253PGG8.pdf" H 7950 3850 50  0001 L CNN
+F 4 "TSSOP 4.4 MM  0.65MM PITCH" H 7950 3750 50  0001 L CNN "Description"
+F 5 "1.2" H 7950 3650 50  0001 L CNN "Height"
+F 6 "972-74CBTLV3253PGG8" H 7950 3550 50  0001 L CNN "Mouser Part Number"
+F 7 "https://www.mouser.com/Search/Refine.aspx?Keyword=972-74CBTLV3253PGG8" H 7950 3450 50  0001 L CNN "Mouser Price/Stock"
+F 8 "IDT" H 7950 3350 50  0001 L CNN "Manufacturer_Name"
+F 9 "74CBTLV3253PGG8" H 7950 3250 50  0001 L CNN "Manufacturer_Part_Number"
+	1    7000 3850
+	0    1    1    0
+$EndComp
+$Comp
+L downloaded:74CBTLV3253PGG8 IC4
+U 1 1 62A7A798
+P 8300 3850
+F 0 "IC4" V 8804 3978 50  0000 L CNN
+F 1 "74CBTLV3253PGG8" V 8900 3200 50  0000 L CNN
+F 2 "SamacSys_Parts:SOP65P640X120-16N" H 9250 3950 50  0001 L CNN
+F 3 "https://componentsearchengine.com/Datasheets/1/74CBTLV3253PGG8.pdf" H 9250 3850 50  0001 L CNN
+F 4 "TSSOP 4.4 MM  0.65MM PITCH" H 9250 3750 50  0001 L CNN "Description"
+F 5 "1.2" H 9250 3650 50  0001 L CNN "Height"
+F 6 "972-74CBTLV3253PGG8" H 9250 3550 50  0001 L CNN "Mouser Part Number"
+F 7 "https://www.mouser.com/Search/Refine.aspx?Keyword=972-74CBTLV3253PGG8" H 9250 3450 50  0001 L CNN "Mouser Price/Stock"
+F 8 "IDT" H 9250 3350 50  0001 L CNN "Manufacturer_Name"
+F 9 "74CBTLV3253PGG8" H 9250 3250 50  0001 L CNN "Manufacturer_Part_Number"
+	1    8300 3850
+	0    1    1    0
+$EndComp
+$Comp
+L downloaded:74CBTLV3253PGG8 IC3
+U 1 1 62A7D074
+P 8300 2450
+F 0 "IC3" V 8804 2578 50  0000 L CNN
+F 1 "74CBTLV3253PGG8" V 8850 1800 50  0000 L CNN
+F 2 "SamacSys_Parts:SOP65P640X120-16N" H 9250 2550 50  0001 L CNN
+F 3 "https://componentsearchengine.com/Datasheets/1/74CBTLV3253PGG8.pdf" H 9250 2450 50  0001 L CNN
+F 4 "TSSOP 4.4 MM  0.65MM PITCH" H 9250 2350 50  0001 L CNN "Description"
+F 5 "1.2" H 9250 2250 50  0001 L CNN "Height"
+F 6 "972-74CBTLV3253PGG8" H 9250 2150 50  0001 L CNN "Mouser Part Number"
+F 7 "https://www.mouser.com/Search/Refine.aspx?Keyword=972-74CBTLV3253PGG8" H 9250 2050 50  0001 L CNN "Mouser Price/Stock"
+F 8 "IDT" H 9250 1950 50  0001 L CNN "Manufacturer_Name"
+F 9 "74CBTLV3253PGG8" H 9250 1850 50  0001 L CNN "Manufacturer_Part_Number"
+	1    8300 2450
+	0    1    1    0
+$EndComp
 $EndSCHEMATC
